File: Sensor/EEE3088F Micromouse.kicad_sch (KiCad schematic)
At the start: 36 parts, among them Q1 2N3904, Q3 2N3904

Commit message: Add files via upload
PROJECT FILES AS AT 24/03/2024
Parts:
- removed D10, D11, D12, D13, D8, D9: TSAL4400, LED_THT:LED_D3.0mm_IRBlack, symbol LED:TSAL4400
- removed D2, D3, D6, D7: SFH213FA, symbol Device:D_Photo
- removed D4, D5: (no value), symbol Device:D_Photo
- removed Q1, Q3: 2N3904, Package_TO_SOT_THT:TO-92_Inline, symbol Transistor_BJT:2N3904
- removed Q2: (no value), symbol Transistor_BJT:2N3904
- removed TP6: TestPoint, symbol Connector:TestPoint
- added C1, C2, C3: 10nF, Capacitor_SMD:C_0805_2012Metric, symbol Device:C_Small
- added D1, D3, D4: IR204A/H60, nicroomouse:IR204_D3.0mm_Horizontal_O1.27mm_Z2.0mm, symbol LED:IR204A
- added JP6: jumper6, Jumper:SolderJumper-2_P1.3mm_Open_Pad1.0x1.5mm, symbol Jumper:Jumper_2_Open
- added JP7: jumper7, Jumper:SolderJumper-2_P1.3mm_Open_Pad1.0x1.5mm, symbol Jumper:Jumper_2_Open
- added JP8: jumper8, Jumper:SolderJumper-2_P1.3mm_Open_Pad1.0x1.5mm, symbol Jumper:Jumper_2_Open
- added Q1, Q2, Q3: AO3400A, Package_TO_SOT_SMD:SOT-23, symbol Transistor_FET:AO3400A
- added Q4, Q5, Q6: PT204-6B, symbol Device:Q_Photo_NPN_EC
- added R10, R8: 47, Resistor_SMD:R_0805_2012Metric, symbol Device:R_Small_US
- added R11, R13, R15: 10k, Resistor_SMD:R_0805_2012Metric, symbol Device:R_Small_US
- added R12, R14, R16: 15k, Resistor_SMD:R_0805_2012Metric, symbol Device:R_Small_US
- added R17, R18: 33k, Resistor_SMD:R_0805_2012Metric, symbol Device:R_Small_US
- added R2: 180, Resistor_SMD:R_0805_2012Metric, symbol Device:R_Small_US
- added R9: 12k, Resistor_SMD:R_0805_2012Metric, symbol Device:R_Small_US
- added TP4: output_R, TestPoint:TestPoint_Pad_D3.0mm, symbol Connector:TestPoint
- added U1, U2, U3: (no value), nicroomouse:SOIC127P599X175-8N, symbol Amplifier_Operational:OP07
- D2: renamed from D1; value LED -> (none)
- J1: value (none) -> Conn_02x14_Odd_Even; footprint (none) -> Connector_PinHeader_2.54mm:PinHeader_2x14_P2.54mm_Vertical
- JP1: value Jumper_2_Open -> jumper1; footprint (none) -> Jumper:SolderJumper-2_P1.3mm_Open_Pad1.0x1.5mm
- JP2: value (none) -> jumper2; footprint (none) -> Jumper:SolderJumper-2_P1.3mm_Open_Pad1.0x1.5mm
- JP3: value Jumper_2_Open -> jumper3; footprint (none) -> Jumper:SolderJumper-2_P1.3mm_Open_Pad1.0x1.5mm
- JP4: value Jumper_2_Open -> jumper4; footprint (none) -> Jumper:SolderJumper-2_P1.3mm_Open_Pad1.0x1.5mm
- JP5: value Jumper_2_Open -> jumper5; footprint (none) -> Jumper:SolderJumper-2_P1.3mm_Open_Pad1.0x1.5mm
- JP9: renamed from JP6; value (none) -> jumper9; footprint (none) -> Jumper:SolderJumper-2_P1.3mm_Open_Pad1.0x1.5mm
- R1: value R_Small_US -> 150; footprint (none) -> Resistor_SMD:R_0805_2012Metric
- R19: renamed from R2; value R_Small_US -> 33k; footprint (none) -> Resistor_SMD:R_0805_2012Metric
- R3: value (none) -> 12k; footprint (none) -> Resistor_SMD:R_0805_2012Metric
- R4, R7: value R_Small_US -> 180; footprint (none) -> Resistor_SMD:R_0805_2012Metric
- R5: value R_Small_US -> 47; footprint (none) -> Resistor_SMD:R_0805_2012Metric
- R6: value R_Small_US -> 12k; footprint (none) -> Resistor_SMD:R_0805_2012Metric
- TP1, TP3: footprint (none) -> TestPoint:TestPoint_Pad_D3.0mm
- TP2: value (none) -> TestPoint; footprint (none) -> TestPoint:TestPoint_Pad_D3.0mm
- TP5: value (none) -> output_F; footprint (none) -> TestPoint:TestPoint_Pad_D3.0mm
- TP6: renamed from TP4; value TestPoint -> output_L; footprint (none) -> TestPoint:TestPoint_Pad_D3.0mm
Connections:
- net +3V3: now also C1.1, C2.1, C3.1, D1.2 (A), D3.2 (A), D4.2 (A), Q4.2 (C), Q5.2 (C), Q6.2 (C); no longer JP1.2 (B), JP2.2 (B), JP3.2 (B), JP4.1 (A), JP5.1 (A), JP9.1 (A)
- net +BATT: now also U1.7 (V+), U2.7 (V+), U3.7 (V+)
- net AB0: now also U1.2 (-), U1.6
- net GND: now also C1.2, C2.2, C3.2, R10.2, R17.2, R18.2, R8.2, R9.2, U1.4 (V-), U2.4 (V-), U3.4 (V-); no longer R4.2, R7.2
- net PA3: now also U2.2 (-), U2.6
- net PA4: now also U3.2 (-), U3.6
- net PE10: now also R4.1
- net PE14: now also R7.1
- net PE8: now also R2.1
- net at R5.1: now also JP2.2 (B), TP1.1, Q1.2 (S)
- net at JP4.2 (B): now also TP2.1, Q2.2 (S), R8.1
- net at R3.1: now also Q1.1 (G), R2.2; no longer TP5.1
- net at TP3.1: now also JP6.2 (B), Q3.2 (S), R10.1
- net at JP3.1 (A): now also Q2.3 (D)
- net OutputL: now reaches R19.1, TP6.1
- net OutputL: now also JP9.2 (B), R15.2, U3.3 (+)
- net at R6.1: now also R4.2, Q2.1 (G)
- net at JP1.1 (A): now also Q1.3 (D)
- net at JP5.2 (B): now also D4.1 (K), JP6.1 (A)
- net at JP2.1 (A): now also JP1.2 (B), D1.1 (K)
- new net: Q6.1 (E), R15.1, R16.1
- new net: JP9.1 (A), R16.2
- new net: Q4.1 (E), R11.1, R12.1
- new net: JP7.1 (A), R12.2
- new net: D3.1 (K), JP3.2 (B), JP4.1 (A)
- new net: JP8.1 (A), R14.2
- new net: Q5.1 (E), R13.1, R14.1
- new net: Q3.1 (G), R7.2, R9.1
- new net: JP5.1 (A), Q3.3 (D)
- new net OutputF: JP8.2 (B), R13.2, R18.1, TP5.1, U2.3 (+)
- new net OutputR: JP7.2 (B), R11.2, R17.1, TP4.1, U1.3 (+)
- no-connect marks 0 -> 6
Other:
- note added: "Buffering"
- title: (none) -> Micromouse Schematic
- moved on the sheet: JP9, R19, TP6
